Commit message: multi robot, namespacing, SHARED MAP added and working

File: p2os/p2os_urdf/defs/pioneer3at.xacro (robot description, xacro)
@@ -5,17 +5,9 @@
        xmlns:xacro="http://ros.org/wiki/xacro"
 name="pioneer3at">
-<!--
-        <include filename="$(find p2os_urdf)/defs/pioneer3at_body.xacro"/>
-        <include filename="$(find p2os_urdf)/defs/hokuyo_utm30lx.urdf.xacro"/>
--->
-  <xacro:include filename="$(find p2os_urdf)/defs/pioneer3at_body.xacro"/>
-  <xacro:include filename="$(find p2os_urdf)/defs/hokuyo_utm30lx.urdf.xacro"/>
-  <xacro:include filename="$(find p2os_urdf)/defs/camera_rc2016.urdf.xacro"/>
-  <xacro:hokuyo_utm30lx name="laser" parent="base_link" ros_topic="scan" update_rate="30" ray_count="1040" min_angle="175" max_angle="-175" >
+<include filename="$(find p2os_urdf)/defs/pioneer3at_body.xacro"/>
+<include filename="$(find p2os_urdf)/defs/hokuyo_utm30lx.urdf.xacro"/>
+<xacro:hokuyo_utm30lx name="laser" parent="base_link" ros_topic="scan" update_rate="30" ray_count="1040" min_angle="130" max_angle="-130" >
     <origin xyz="0.13 0 0.32" rpy="0 0 0"/>
   </xacro:hokuyo_utm30lx>
-  <xacro:camera_rc2016 name="camera" parent="base_link" ros_topic="camera" update_rate="30" height="0.09">
-    <origin xyz="0.13 0 0.32" rpy="0 0 0"/>
-  </xacro:camera_rc2016>
 <xacro:p3at_front suffix="left" reflect="1"/>
 <xacro:p3at_front suffix="right" reflect="-1"/>
