Commit message: xacro model fixed

File: p2os/p2os_urdf/defs-old/pioneer3at_body.xacro (robot description, xacro)
@@ -8,9 +8,9 @@
 	<link name="base_link">
 		<inertial>
-			<mass value="10.0"/>
-			<origin xyz="0 0 0.177"/>
-			<inertia ixx="0.3338" ixy="0.0" ixz="0.0"
-				 iyy="0.4783" iyz="0.0"
-				 izz="0.3338"/>
+		  <mass value="14.0"/>
+		  <origin xyz="0 0 0.177"/>
+		  <inertia ixx="0.14711667" ixy="0.0" ixz="0.0"
+			iyy="0.334951167" iyz="0.0"
+			izz="0.3978345"/>
 		</inertial>
 		<visual name="base_visual">
@@ -36,9 +36,9 @@
 	<link name="top_plate">
 		<inertial>
-			<mass value="0.1"/>
+			<mass value="3.0"/>
 			<origin xyz="-0.025 0 -0.223"/>
-			<inertia ixx="1.0" ixy="0.0" ixz="0.0"
-				 iyy="1.0" iyz="0.0"
- 				izz="1.0"/>
+			  <inertia ixx="0.14711667" ixy="0.0" ixz="0.0"
+				iyy="0.334951167" iyz="0.0"
+				izz="0.3978345"/>
 		</inertial>
 		<visual name="base_visual">
@@ -69,8 +69,9 @@
 	<link name="front_sonar">
 		<inertial>
-			<mass value="0.1"/>
+			<mass value="2.0"/>
 			<origin xyz="0 0 0"/>
-			<inertia ixx="1.0" ixy="0.0" ixz="0.0"
-				 iyy="1.0" iyz="0.0" izz="1.0"/>
+			  <inertia ixx="0.14711667" ixy="0.0" ixz="0.0"
+				iyy="0.334951167" iyz="0.0"
+				izz="0.3978345"/>
 		</inertial>
 		<visual name="base_visual">
@@ -100,8 +101,9 @@
 	<link name="back_sonar">
 		<inertial>
-			<mass value="0.1"/>
+			<mass value="2.0"/>
 			<origin xyz="0 0 0"/>
-			<inertia ixx="1.0" ixy="0.0" ixz="0.0"
-				 iyy="1.0" iyz="0.0" izz="1.0"/>
+			  <inertia ixx="0.14711667" ixy="0.0" ixz="0.0"
+				iyy="0.334951167" iyz="0.0"
+				izz="0.3978345"/>
 		</inertial>
 		<visual name="base_visual">
@@ -133,8 +135,8 @@
 	<link name="p3at_front_${suffix}_axle">
 		<inertial>
-			<mass value="0.1"/>
-			<origin xyz="0 0 0"/>
-			<inertia ixx="1.0" ixy="0.0" ixz="0.0"
-				 iyy="1.0" iyz="0.0" izz="1.0"/>
+      		  <mass value="1.5"/>
+				<origin xyz="0 0 0"/>
+				<inertia ixx="0.005240625" ixy="0" ixz="0"
+				iyy="0.005240625" iyz="0" izz="0.009075"/>
   	 	</inertial>
 	<visual name="base_visual">
@@ -164,8 +166,8 @@
 	<link name="p3at_front_${suffix}_hub">
 		<inertial>
-			<mass value="0.1"/>
-			<origin xyz="0 0 0"/>
-			<inertia ixx="1.0" ixy="0.0" ixz="0.0"
-				 iyy="1.0" iyz="0.0" izz="1.0"/>
+		  <mass value="1.5"/>
+		  <origin xyz="0 0 0"/>
+		  <inertia ixx="0.005240625" ixy="0" ixz="0"
+			iyy="0.005240625" iyz="0" izz="0.009075"/>
   	 	</inertial>
 	<visual name="base_visual">
@@ -195,8 +197,8 @@
 	<link name="p3at_front_${suffix}_wheel">
 		<inertial>
-			<mass value="0.5"/>
-			<origin xyz="0 0 0"/>
-			<inertia ixx="0.012411765597" ixy="0" ixz="0"
-         iyy="0.015218160428" iyz="0" izz="0.011763977943"/>
+		  <mass value="1.5"/>
+		  <origin xyz="0 0 0"/>
+		  <inertia ixx="0.005240625" ixy="0" ixz="0"
+			iyy="0.005240625" iyz="0" izz="0.009075"/>
       </inertial>
 	<visual name="base_visual">
@@ -234,8 +236,8 @@
 	<link name="p3at_back_${suffix}_axle">
 		<inertial>
-			<mass value="0.1"/>
-			<origin xyz="0 0 0"/>
-			<inertia ixx="1.0" ixy="0.0" ixz="0.0"
-				 iyy="1.0" iyz="0.0" izz="1.0"/>
+		  <mass value="1.5"/>
+		  <origin xyz="0 0 0"/>
+		  <inertia ixx="0.005240625" ixy="0" ixz="0"
+			iyy="0.005240625" iyz="0" izz="0.009075"/>
   	 	</inertial>
 	<visual name="base_visual">
@@ -265,8 +267,8 @@
 	<link name="p3at_back_${suffix}_hub">
 		<inertial>
-			<mass value="0.1"/>
-			<origin xyz="0 0 0"/>
-			<inertia ixx="1.0" ixy="0.0" ixz="0.0"
-				 iyy="1.0" iyz="0.0" izz="1.0"/>
+		  <mass value="1.5"/>
+		  <origin xyz="0 0 0"/>
+		  <inertia ixx="0.005240625" ixy="0" ixz="0"
+			iyy="0.005240625" iyz="0" izz="0.009075"/>
   	 	</inertial>
 	<visual name="base_visual">
@@ -294,8 +296,8 @@
 	<link name="p3at_back_${suffix}_wheel">
 		<inertial>
-			<mass value="0.5"/>
-			<origin xyz="0 0 0"/>
-			<inertia ixx="0.012411765597" ixy="0" ixz="0"
-         iyy="0.015218160428" iyz="0" izz="0.011763977943"/>
+		  <mass value="1.5"/>
+		  <origin xyz="0 0 0"/>
+		  <inertia ixx="0.005240625" ixy="0" ixz="0"
+			iyy="0.005240625" iyz="0" izz="0.009075"/>
       </inertial>
 	<visual name="base_visual">

File: p2os/p2os_urdf/defs-old/pioneer3at_body2.xacro (robot description, xacro)
@@ -8,9 +8,9 @@
 	<link name="base_link">
 		<inertial>
-			<mass value="10.0"/>
-			<origin xyz="0 0 0.177"/>
-			<inertia ixx="0.3338" ixy="0.0" ixz="0.0"
-				 iyy="0.4783" iyz="0.0"
-				 izz="0.3338"/>
+		  <mass value="14.0"/>
+		  <origin xyz="0 0 0.177"/>
+		  <inertia ixx="0.14711667" ixy="0.0" ixz="0.0"
+			iyy="0.334951167" iyz="0.0"
+			izz="0.3978345"/>
 		</inertial>
 		<visual name="base_visual">
@@ -36,9 +36,9 @@
 	<link name="top_plate">
 		<inertial>
-			<mass value="0.1"/>
+			<mass value="3.0"/>
 			<origin xyz="-0.025 0 -0.223"/>
-			<inertia ixx="1.0" ixy="0.0" ixz="0.0"
-				 iyy="1.0" iyz="0.0"
- 				izz="1.0"/>
+			  <inertia ixx="0.14711667" ixy="0.0" ixz="0.0"
+				iyy="0.334951167" iyz="0.0"
+				izz="0.3978345"/>
 		</inertial>
 		<visual name="base_visual">
@@ -69,8 +69,9 @@
 	<link name="front_sonar">
 		<inertial>
-			<mass value="0.1"/>
+			<mass value="2.0"/>
 			<origin xyz="0 0 0"/>
-			<inertia ixx="1.0" ixy="0.0" ixz="0.0"
-				 iyy="1.0" iyz="0.0" izz="1.0"/>
+			  <inertia ixx="0.14711667" ixy="0.0" ixz="0.0"
+				iyy="0.334951167" iyz="0.0"
+				izz="0.3978345"/>
 		</inertial>
 		<visual name="base_visual">
@@ -100,8 +101,9 @@
 	<link name="back_sonar">
 		<inertial>
-			<mass value="0.1"/>
+			<mass value="2.0"/>
 			<origin xyz="0 0 0"/>
-			<inertia ixx="1.0" ixy="0.0" ixz="0.0"
-				 iyy="1.0" iyz="0.0" izz="1.0"/>
+			  <inertia ixx="0.14711667" ixy="0.0" ixz="0.0"
+				iyy="0.334951167" iyz="0.0"
+				izz="0.3978345"/>
 		</inertial>
 		<visual name="base_visual">
@@ -133,8 +135,8 @@
 	<link name="p3at_front_${suffix}_axle">
 		<inertial>
-			<mass value="0.1"/>
-			<origin xyz="0 0 0"/>
-			<inertia ixx="1.0" ixy="0.0" ixz="0.0"
-				 iyy="1.0" iyz="0.0" izz="1.0"/>
+      		  <mass value="1.5"/>
+				<origin xyz="0 0 0"/>
+				<inertia ixx="0.005240625" ixy="0" ixz="0"
+				iyy="0.005240625" iyz="0" izz="0.009075"/>
   	 	</inertial>
 	<visual name="base_visual">
@@ -164,8 +166,8 @@
 	<link name="p3at_front_${suffix}_hub">
 		<inertial>
-			<mass value="0.1"/>
-			<origin xyz="0 0 0"/>
-			<inertia ixx="1.0" ixy="0.0" ixz="0.0"
-				 iyy="1.0" iyz="0.0" izz="1.0"/>
+		  <mass value="1.5"/>
+		  <origin xyz="0 0 0"/>
+		  <inertia ixx="0.005240625" ixy="0" ixz="0"
+			iyy="0.005240625" iyz="0" izz="0.009075"/>
   	 	</inertial>
 	<visual name="base_visual">
@@ -195,8 +197,8 @@
 	<link name="p3at_front_${suffix}_wheel">
 		<inertial>
-			<mass value="0.5"/>
-			<origin xyz="0 0 0"/>
-			<inertia ixx="0.012411765597" ixy="0" ixz="0"
-         iyy="0.015218160428" iyz="0" izz="0.011763977943"/>
+		  <mass value="1.5"/>
+		  <origin xyz="0 0 0"/>
+		  <inertia ixx="0.005240625" ixy="0" ixz="0"
+			iyy="0.005240625" iyz="0" izz="0.009075"/>
       </inertial>
 	<visual name="base_visual">
@@ -234,8 +236,8 @@
 	<link name="p3at_back_${suffix}_axle">
 		<inertial>
-			<mass value="0.1"/>
-			<origin xyz="0 0 0"/>
-			<inertia ixx="1.0" ixy="0.0" ixz="0.0"
-				 iyy="1.0" iyz="0.0" izz="1.0"/>
+		  <mass value="1.5"/>
+		  <origin xyz="0 0 0"/>
+		  <inertia ixx="0.005240625" ixy="0" ixz="0"
+			iyy="0.005240625" iyz="0" izz="0.009075"/>
   	 	</inertial>
 	<visual name="base_visual">
@@ -265,8 +267,8 @@
 	<link name="p3at_back_${suffix}_hub">
 		<inertial>
-			<mass value="0.1"/>
-			<origin xyz="0 0 0"/>
-			<inertia ixx="1.0" ixy="0.0" ixz="0.0"
-				 iyy="1.0" iyz="0.0" izz="1.0"/>
+		  <mass value="1.5"/>
+		  <origin xyz="0 0 0"/>
+		  <inertia ixx="0.005240625" ixy="0" ixz="0"
+			iyy="0.005240625" iyz="0" izz="0.009075"/>
   	 	</inertial>
 	<visual name="base_visual">
@@ -294,8 +296,8 @@
 	<link name="p3at_back_${suffix}_wheel">
 		<inertial>
-			<mass value="0.5"/>
-			<origin xyz="0 0 0"/>
-			<inertia ixx="0.012411765597" ixy="0" ixz="0"
-         iyy="0.015218160428" iyz="0" izz="0.011763977943"/>
+		  <mass value="1.5"/>
+		  <origin xyz="0 0 0"/>
+		  <inertia ixx="0.005240625" ixy="0" ixz="0"
+			iyy="0.005240625" iyz="0" izz="0.009075"/>
       </inertial>
 	<visual name="base_visual">
@@ -356,5 +358,5 @@
     <wheelSeparation>0.4</wheelSeparation>
     <wheelDiameter>0.215</wheelDiameter>
-    <robotBaseFrame>base_link	</robotBaseFrame>
+    <robotBaseFrame>base_link</robotBaseFrame>
     <torque>200</torque>
     <topicName>cmd_vel</topicName>

File: p2os/p2os_urdf/defs-old/pioneer3at_body4.xacro (robot description, xacro)
@@ -351,5 +351,5 @@
   <plugin name="skid_steer_drive_controller" filename="libgazebo_ros_skid_steer_drive.so">
     <updateRate>100.0</updateRate>
-    <robotNamespace>robot3</robotNamespace>
+    <robotNamespace>robot4</robotNamespace>
     <leftFrontJoint>p3at_front_left_wheel_joint</leftFrontJoint>
     <rightFrontJoint>p3at_front_right_wheel_joint</rightFrontJoint>
